File: OpenStage_PCB/OpenStage.brd (EAGLE design)
At the start: 167 x 134.6 mm, 65 parts, among them J1 M8S-04PFFR-SF8001, J3 M8S-04PFFR-SF8001, J4 M8S-04PFFR-SF8001, J5 M8S-04PFFR-SF8001, M1 STEPPER_DRIVER, M2 STEPPER_DRIVER, M3 STEPPER_DRIVER, M4 STEPPER_DRIVER, U2 ARDUINO_SHIELD

Commit message: Generate gerbers for new PCB
Connections:
- removed net QS+5V: C6.P$2, C7.P$1, R15.1, R16.1, U$4.16, U2.5V
- new net N$3: U2.5V
- net +5V: now also C6.P$2, C7.P$1, R15.1, R16.1, U$4.16
Routing:
- net +5V: track 335.4 -> 496.2 mm
- net QS+5V: track 73.4 -> 0.00 mm
Changed lines of the file:
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@@
 Rob Campbell, 2014
 </text>
-<text x="24.765" y="79.375" size="1.778" layer="25">CH 3</text>
-<text x="45.085" y="79.375" size="1.778" layer="25">CH 4</text>
-<text x="24.765" y="104.14" size="1.778" layer="25">CH 1</text>
-<text x="45.085" y="104.14" size="1.778" layer="25">CH 2</text>
+<text x="27.765" y="81.575" size="1.778" layer="25" rot="SR180" align="center">CH 3</text>
+<text x="48.085" y="81.375" size="1.778" layer="25" rot="SR180" align="center">CH 4</text>
+<text x="27.565" y="105.14" size="1.778" layer="25" rot="SR180" align="center">CH 1</text>
+<text x="47.885" y="105.14" size="1.778" layer="25" rot="SR180" align="center">CH 2</text>
 <circle x="6.985" y="116.84" radius="0.635" width="0.8128" layer="26"/>
 <wire x1="6.985" y1="116.84" x2="12.7" y2="116.84" width="0.8128" layer="26"/>
@@
 <contactref element="PCB2" pad="5V"/>
 <wire x1="128.5875" y1="44.45" x2="131.445" y2="44.45" width="0.3" layer="1"/>
-<wire x1="131.445" y1="44.45" x2="137.795" y2="44.45" width="0.3" layer="1"/>
+<wire x1="131.445" y1="44.45" x2="135" y2="44.45" width="0.3" layer="1"/>
+<contactref element="R15" pad="1"/>
+<contactref element="R16" pad="1"/>
+<wire x1="137.795" y1="44.45" x2="135" y2="44.45" width="0.3" layer="1"/>
+<wire x1="135" y1="44.45" x2="133.8" y2="43.25" width="0.2" layer="1"/>
+<wire x1="133.8" y1="43.25" x2="133.8" y2="22.6" width="0.2" layer="1"/>
+<wire x1="133.8" y1="22.6" x2="129.2" y2="18" width="0.2" layer="1"/>
+<wire x1="66.81616875" y1="12.7778" x2="66.79396875" y2="12.8" width="0.2" layer="1"/>
+<wire x1="129.2" y1="18" x2="75" y2="18" width="0.2" layer="1"/>
+<wire x1="75" y1="18" x2="69.7778" y2="12.7778" width="0.2" layer="1"/>
+<wire x1="69.7778" y1="12.7778" x2="66.81616875" y2="12.7778" width="0.2" layer="1"/>
+<wire x1="56" y1="14" x2="42.6" y2="14" width="0.2" layer="1"/>
+<wire x1="66.79396875" y1="12.8" x2="57.2" y2="12.8" width="0.2" layer="1"/>
+<wire x1="57.2" y1="12.8" x2="56" y2="14" width="0.2" layer="1"/>
+<contactref element="U$4" pad="16"/>
+<contactref element="C6" pad="P$2"/>
+<contactref element="C7" pad="P$1"/>
+<wire x1="36.83" y1="19.685" x2="26.72841875" y2="19.685" width="0.3048" layer="16"/>
+<wire x1="26.72841875" y1="19.685" x2="26.71" y2="15.875" width="0.3048" layer="16"/>
+<wire x1="23.6" y1="16" x2="26.585" y2="16" width="0.2" layer="1"/>
+<wire x1="26.585" y1="16" x2="26.71" y2="15.875" width="0.2" layer="1"/>
+<wire x1="42.6" y1="14" x2="36.915" y2="19.685" width="0.2" layer="1"/>
+<wire x1="36.83" y1="19.685" x2="36.915" y2="19.685" width="0.2" layer="1"/>
+<wire x1="36.83" y1="19.685" x2="36.195" y2="20.32" width="0.2" layer="1"/>
+<wire x1="36.195" y1="20.32" x2="36.195" y2="22.2" width="0.2" layer="1"/>
+<wire x1="36.195" y1="22.2" x2="36.195" y2="24.1905" width="0.2" layer="1"/>
+<wire x1="31.71" y1="22.225" x2="36.17" y2="22.225" width="0.2" layer="1"/>
+<wire x1="36.17" y1="22.225" x2="36.195" y2="22.2" width="0.2" layer="1"/>
+<wire x1="23.6" y1="16" x2="23.495" y2="16.105" width="0.2" layer="1"/>
+<wire x1="23.495" y1="16.105" x2="23.495" y2="24.1905" width="0.2" layer="1"/>
 </signal>
 <signal name="A15">
@@
 <wire x1="46.6755" y1="26.9905" x2="46.99" y2="27.305" width="0.3048" layer="1"/>
 </signal>
-<signal name="QS+5V">
-<contactref element="R15" pad="1"/>
-<contactref element="R16" pad="1"/>
-<wire x1="23.495" y1="24.1905" x2="23.495" y2="16" width="0.3048" layer="1"/>
-<wire x1="36.195" y1="24.1905" x2="31.8105" y2="24.1905" width="0.3048" layer="1"/>
-<wire x1="31.8105" y1="24.1905" x2="31.75" y2="24.13" width="0.3048" layer="1"/>
-<contactref element="U$4" pad="16"/>
-<contactref element="C6" pad="P$2"/>
-<contactref element="C7" pad="P$1"/>
-<wire x1="36.83" y1="19.685" x2="26.72841875" y2="19.685" width="0.3048" layer="16"/>
-<wire x1="26.72841875" y1="19.685" x2="26.71" y2="15.875" width="0.3048" layer="16"/>
-<wire x1="34.29" y1="22.225" x2="33.8" y2="22.225" width="0.3048" layer="16"/>
-<wire x1="34.29" y1="22.225" x2="36.83" y2="19.685" width="0.3048" layer="16"/>
-<contactref element="U2" pad="5V"/>
-<wire x1="67.31" y1="31.75" x2="57.76" y2="22.2" width="0.3" layer="1"/>
-<wire x1="39.345" y1="22.2" x2="36.83" y2="19.685" width="0.3" layer="1"/>
-<wire x1="57.76" y1="22.2" x2="39.345" y2="22.2" width="0.3" layer="1"/>
-<wire x1="23.495" y1="16" x2="26.585" y2="16" width="0.2" layer="1"/>
-<wire x1="26.585" y1="16" x2="26.71" y2="15.875" width="0.2" layer="1"/>
-<wire x1="33.8" y1="22.225" x2="31.71" y2="22.225" width="0.2" layer="16"/>
-<wire x1="31.75" y1="24.13" x2="31.71" y2="24.09" width="0.2" layer="1"/>
-<wire x1="31.71" y1="24.09" x2="31.71" y2="22.225" width="0.2" layer="1"/>
-</signal>
 <signal name="A14">
 <contactref element="PCB2" pad="A14"/>
@@
 <wire x1="139.065" y1="13.205" x2="139.065" y2="9.525" width="0.2" layer="16"/>
 </signal>
+<signal name="N$3">
+<contactref element="U2" pad="5V"/>
+</signal>
 </signals>
